File: pcb/kicad/abadi-motherboard.kicad_pcb (KiCad board)
At the start: 2 copper layers, 100 x 100 mm, 38 parts, among them J1 ESP32-S3 row 1 (3V3 RST 4 5 .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, J3 ESP32-S3 row 2 (GND TX RX 1 2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

Commit message: Motherboard v5: DRV8833 two rows of 6 holes, screen pin order, ratings, stitching vias
DRV8833 (HW-627) footprints now follow the owner's reading of the module: top
row IN1 IN2 VCC GND IN3 IN4 (VCC = battery), bottom row (white plug side) EEP
OUT1 OUT2 OUT3 OUT4 ULT, with the pin names printed. Screen headers follow the
screens' own order CS DC RST SDA SCL VCC GND. Capacitor ratings are printed on
the board and listed in the parts list, which now says what to buy for every
footprint. Outline trimmed so the Gerber extents are exactly 100.0 x 100.0 mm.
30 ground stitching vias tie the two ground pours together. New shopping list
(including off-board power parts and first power-up steps); README rewritten.

Routed on 2 layers: KiCad DRC 0 errors / 0 unconnected; independent Gerber
audit 0 shorts / 0 opens (211 plated holes matched). Row gap and alignment of
the DRV8833 holes still to be confirmed on the real module.

Co-Authored-By: Claude Sonnet 5.5 <noreply@anthropic.com>
Claude-Session: https://claude.ai/code/session_01FTMr77tNTaQwRQC74wgVC1
Parts:
- moved DRVA 1.01 mm to (138.2, 103.0)
- moved DRVB 1.01 mm to (164.2, 103.0)
- moved RD2a 0.80 mm to (181.5, 92.5)
- moved RD2b 0.80 mm to (186.5, 92.5)
- moved SON2 0.80 mm to (180.0, 89.0)
- moved RD1a 0.60 mm to (168.4, 92.5)
- moved RD1b 0.60 mm to (173.4, 92.5)
- moved SON1 0.60 mm to (166.9, 89.0)
- moved RLY3H 0.40 mm to (156.2, 89.0)
- moved RLY2H 0.20 mm to (145.6, 89.0)
- moved SCR_L 0.20 mm to (137.0, 54.2)
- moved SCR_R 0.20 mm to (155.0, 54.2)
- moved SPARE 0.20 mm to (173.2, 54.2)
- moved UART 0.20 mm to (148.2, 93.4)
Connections:
- DRVA pad 10: M2B -> M2A
- DRVA pad 3: IN3A -> VBAT
- DRVA pad 4: IN4A -> GND
- DRVA pad 5: GND -> IN3A
- DRVA pad 6: VBAT -> IN4A
- DRVA pad 7: M1A -> (no net)
- DRVA pad 8: M1B -> M1A
- DRVA pad 9: M2A -> M1B
- DRVB pad 10: M4B -> M4A
- DRVB pad 3: IN3B -> VBAT
- DRVB pad 4: IN4B -> GND
- DRVB pad 5: GND -> IN3B
- DRVB pad 6: VBAT -> IN4B
- DRVB pad 7: M3A -> (no net)
- DRVB pad 8: M3B -> M3A
- DRVB pad 9: M4A -> M3B
- SCR_L pad 1: RAILC -> CS_L
- SCR_L pad 2: GND -> LCD_DC
- SCR_L pad 3: CS_L -> LCD_RST
- SCR_L pad 4: LCD_RST -> MOSI
- SCR_L pad 5: LCD_DC -> SCK
- SCR_L pad 6: MOSI -> RAILC
- SCR_L pad 7: SCK -> GND
- SCR_R pad 1: RAILC -> CS_R
- SCR_R pad 2: GND -> LCD_DC
- SCR_R pad 3: CS_R -> LCD_RST
- SCR_R pad 4: LCD_RST -> MOSI
- SCR_R pad 5: LCD_DC -> SCK
- SCR_R pad 6: MOSI -> RAILC
- SCR_R pad 7: SCK -> GND
Routing:
- net VBAT: track 97.7 -> 142.6 mm
- net LCD_DC: track 32.8 -> 23.1 mm
- net SCK: track 32.4 -> 41.5 mm, vias 1 -> 0
- net RAILC: track 217.0 -> 225.4 mm
- net IN3B: track 28.6 -> 20.5 mm
- net IN4B: track 28.5 -> 20.5 mm
- net ESP3V3: track 128.1 -> 135.9 mm, vias 0 -> 1
- net CS_R: track 14.7 -> 6.87 mm
- net SPARE38: track 33.2 -> 40.8 mm
- net IN1A: track 29.7 -> 22.3 mm
- net SCL: track 90.4 -> 97.6 mm, vias 1 -> 2
- net CS_L: track 6.74 -> 11.9 mm
- net ECHO1_3V: track 16.2 -> 20.1 mm, vias 0 -> 1
- net IN2B: track 25.2 -> 29.0 mm
- net SPARE3: track 37.3 -> 33.7 mm
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Other:
- board size 100 x 100 mm -> 99.9 x 99.9 mm
- board text added: "ABADI MOTHERBOARD v5 (2L)"
- board text added: "C1 470uF 16V"
- board text added: "C2 100uF 10V"
- board text added: "C3 100n"
- board text added: "C4 100n"
- board text added: "EEP"
- board text added: "OUT1"
- board text added: "OUT2"
- board text added: "OUT3"
- board text added: "OUT4"
- board text added: "ULT"
- board text added: "white plug v"
- board text removed: "ABADI MOTHERBOARD v4 (2L)"
- board text removed: "C1 470uF"
- board text removed: "C2 100uF"
- board text removed: "C3"
- board text removed: "C4"
- board text removed: "M1A"
- board text removed: "M1B"
- board text removed: "M2A"
- board text removed: "M2B"
- board text removed: "M3A"
- board text removed: "M3B"
- board text removed: "M4A"
- board text removed: "M4B"
- board text removed: "VM"
